Commit message: fix: Add `base_footprint` link and joint to correct robot model orientation.

File: Others/palletizer_v1_ws/src/palletizer_v1_description/urdf/palletizer_v1_description.urdf (robot description, URDF)
Before this commit: robot palletizer_v1_description, 8 links, 7 joints
Links:
- added link base_footprint
Joints:
- added joint base_footprint_joint: type fixed, parent base_footprint, child base_link, origin xyz=0 0 0 rpy=1.5708 0 0

Commit message: feat: Add Gazebo differential drive and joint state plugins, wheel friction properties, base link color, and correct wheel joint axes.

File: Others/palletizer_v1_ws/src/palletizer_v1_description/urdf/palletizer_v1_description.urdf (robot description, URDF)
Before this commit: robot palletizer_v1_description, 9 links, 8 joints
Joints:
- joint j1: axis 0 0 -1 -> 0 0 1
- joint j2: axis 0 0 -1 -> 0 0 1

Commit message: fix: correct joint origin and lidar sensor rotations in URDF

File: Others/palletizer_v1_ws/src/palletizer_v1_description/urdf/palletizer_v1_description.urdf (robot description, URDF)
Before this commit: robot palletizer_v1_description, 9 links, 8 joints
Joints:
- joint lidar_joint: origin xyz=-0.044699 0.29873 0.00015762 rpy=0 0 0 -> xyz=-0.044699 0.29873 0.00015762 rpy=1.5708 0 0

Commit message: feat: Rotate base_footprint_joint by 180 degrees and increase odometry, joint states, and lidar update rates to 50Hz.

File: Others/palletizer_v1_ws/src/palletizer_v1_description/urdf/palletizer_v1_description.urdf (robot description, URDF)
Before this commit: robot palletizer_v1_description, 9 links, 8 joints
Joints:
- joint base_footprint_joint: origin xyz=0 0 0 rpy=1.5708 0 0 -> xyz=0 0 0 rpy=1.5708 0 3.14159

Commit message: feat: Add stereo camera and visual odometry support with Gazebo-ROS bridging.

File: Others/palletizer_v1_ws/src/palletizer_v1_description/urdf/palletizer_v1_description.urdf (robot description, URDF)
Before this commit: robot palletizer_v1_description, 9 links, 8 joints
Links:
- added link camera_left_optical_frame
- added link camera_right_optical_frame
Joints:
- added joint camera_left_optical_joint: type fixed, parent camera_link, child camera_left_optical_frame, origin xyz=0 0.06 0 rpy=-1.5708 0 -1.5708
- added joint camera_right_optical_joint: type fixed, parent camera_link, child camera_right_optical_frame, origin xyz=0 -0.06 0 rpy=-1.5708 0 -1.5708

Commit message: fix: Adjust camera and optical frame origins in URDF.

File: Others/palletizer_v1_ws/src/palletizer_v1_description/urdf/palletizer_v1_description.urdf (robot description, URDF)
Before this commit: robot palletizer_v1_description, 11 links, 10 joints
Joints:
- joint camera_joint: origin xyz=-0.23713 0.1899 0.00015762 rpy=0 0 0 -> xyz=-0.23713 0.1899 0.00015762 rpy=3.14159 0 1.5708
- joint camera_left_optical_joint: origin xyz=0 0.06 0 rpy=-1.5708 0 -1.5708 -> xyz=0 0 0.08 rpy=-1.5708 0 -1.5708
- joint camera_right_optical_joint: origin xyz=0 -0.06 0 rpy=-1.5708 0 -1.5708 -> xyz=0 0 -0.08 rpy=-1.5708 0 -1.5708

Commit message: feat: Implement custom visual odometry publishing via a new ROS2 node, replacing the Gazebo pose publisher, and correct camera optical joint origins.

File: Others/palletizer_v1_ws/src/palletizer_v1_description/urdf/palletizer_v1_description.urdf (robot description, URDF)
Before this commit: robot palletizer_v1_description, 11 links, 10 joints
Joints:
- joint camera_left_optical_joint: origin xyz=0 0 0.08 rpy=-1.5708 0 -1.5708 -> xyz=0 0 -0.08 rpy=-1.5708 0 -1.5708
- joint camera_right_optical_joint: origin xyz=0 0 -0.08 rpy=-1.5708 0 -1.5708 -> xyz=0 0 0.08 rpy=-1.5708 0 -1.5708

Commit message: feat: add Sharp IR distance sensor to URDF, configure Gazebo-ROS bridge, and reorient the sensor link.

File: Others/palletizer_v1_ws/src/palletizer_v1_description/urdf/palletizer_v1_description.urdf (robot description, URDF)
Before this commit: robot palletizer_v1_description, 11 links, 10 joints
Joints:
- joint sensors_joint: origin xyz=-0.28745 -0.023774 0.00015762 rpy=0 0 0 -> xyz=-0.28745 -0.023774 0.00015762 rpy=1.5708 0 3.14159
