Commit message: feat: Add ArUco marker mesh and texture, integrate it into `caja1.urdf`, and spawn the box in Gazebo.

File: Others/palletizer_v1_ws/src/palletizer_v1_description/urdf/caja1.urdf (robot description, URDF)
Before this commit: robot caja1, 9 links, 8 joints
Links:
- added link aruco_marker_link; visual mesh filename=package://palletizer_v1_description/meshes/aruco_marker_1.d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
Joints:
- added joint aruco_marker_joint: type fixed, parent base_link_caja, child aruco_marker_link, origin xyz=0.145 0 0.30 rpy=0 0 0

Commit message: fix: update link4 inertial properties with calculated mass and inertia values

File: Others/palletizer_v1_ws/src/palletizer_v1_description/urdf/caja1.urdf (robot description, URDF)
Before this commit: robot caja1, 10 links, 9 joints
Links:
- link link4: mass 0 -> 0.028235

Commit message: feat: Update URDF to define continuous joints with dynamics and add Gazebo friction settings for caster wheels.

File: Others/palletizer_v1_ws/src/palletizer_v1_description/urdf/caja1.urdf (robot description, URDF)
Before this commit: robot caja1, 10 links, 9 joints
Joints:
- joint joint1: limit lower=-3.14159 upper=3.14159 effort=0 velocity=0 -> (none); type revolute -> continuous
- joint joint2: limit lower=-3.14159 upper=3.14159 effort=0 velocity=0 -> (none); type revolute -> continuous
- joint joint3: limit lower=-3.14159 upper=3.14159 effort=0 velocity=0 -> (none); type revolute -> continuous
- joint joint4: limit lower=-3.14159 upper=3.14159 effort=0 velocity=0 -> (none); type revolute -> continuous

Commit message: feat: update caja1 URDF to increase mass and set wheel friction coefficients to zero.

File: Others/palletizer_v1_ws/src/palletizer_v1_description/urdf/caja1.urdf (robot description, URDF)
Before this commit: robot caja1, 10 links, 9 joints
Links:
- link base_link_caja: mass 30 -> 40

Commit message: add: Up aruco, and remove some cluttering and Shelf

File: Others/palletizer_v1_ws/src/palletizer_v1_description/urdf/caja1.urdf (robot description, URDF)
Before this commit: robot caja1, 10 links, 9 joints
Joints:
- joint aruco_marker_joint: origin xyz=0.145 0 0.30 rpy=0 0 0 -> xyz=0.145 0 0.43 rpy=0 0 0
